Commit message: modified effort and pid constants

File: test_legs_urdf/urdf/test_legs_urdf.urdf (robot description, URDF)
Before this commit: robot test_legs_urdf, 13 links, 12 joints
Joints:
- joint LAnkle_pitch: limit lower=-1.57 upper=1.57 effort=0.3 velocity=5 -> lower=-1.57 upper=1.57 effort=1.3 velocity=5
- joint LAnkle_roll: limit lower=-1.57 upper=1.57 effort=0.3 velocity=5 -> lower=-1.57 upper=1.57 effort=1.3 velocity=5
- joint LHip_pitch: limit lower=-1.57 upper=1.57 effort=0.3 velocity=5 -> lower=-1.57 upper=1.57 effort=1.3 velocity=5
- joint LHip_roll: limit lower=-1.57 upper=1.57 effort=0.3 velocity=5 -> lower=-1.57 upper=1.57 effort=1.3 velocity=5
- joint LHip_yaw: limit lower=-1.57 upper=1.57 effort=0.3 velocity=5 -> lower=-1.57 upper=1.57 effort=1.3 velocity=5
- joint LKnee_pitch: limit lower=-1.57 upper=1.57 effort=0.3 velocity=5 -> lower=-1.57 upper=1.57 effort=1.3 velocity=5
- joint RAnkle_pitch: limit lower=-1.57 upper=1.57 effort=0.3 velocity=5 -> lower=-1.57 upper=1.57 effort=1.3 velocity=5
- joint RAnkle_roll: limit lower=-1.57 upper=1.57 effort=0.3 velocity=5 -> lower=-1.57 upper=1.57 effort=1.3 velocity=5
- joint RHip_pitch: limit lower=-1.57 upper=1.57 effort=0.3 velocity=5 -> lower=-1.57 upper=1.57 effort=1.3 velocity=5
- joint RHip_roll: limit lower=-1.57 upper=1.57 effort=0.3 velocity=5 -> lower=-1.57 upper=1.57 effort=1.3 velocity=5
- joint RHip_yaw: limit lower=-1.57 upper=1.57 effort=0.3 velocity=5 -> lower=-1.57 upper=1.57 effort=1.3 velocity=5
- joint RKnee_pitch: limit lower=-1.57 upper=1.57 effort=0.3 velocity=5 -> lower=-1.57 upper=1.57 effort=1.3 velocity=5

Commit message: tuned knee and ankle PID and modified base link mass

File: test_legs_urdf/urdf/test_legs_urdf.urdf (robot description, URDF)
Before this commit: robot test_legs_urdf, 13 links, 12 joints
Links:
- link base_link: mass 0.37523 -> 0.275

Commit message: updated link masses with real values and modified walking gait

File: test_legs_urdf/urdf/test_legs_urdf.urdf (robot description, URDF)
Before this commit: robot test_legs_urdf, 13 links, 12 joints
Links:
- link LAnkle: mass 0.024453 -> 0.02644
- link LFemur: mass 0.053764 -> 0.0839
- link LFoot: mass 0.068473 -> 0.09345
- link LHip: mass 0.049473 -> 0.076
- link LTibia: mass 0.081897 -> 0.13355
- link RAnkle: mass 0.024453 -> 0.02644
- link RFemur: mass 0.053764 -> 0.0839
- link RFoot: mass 0.068473 -> 0.09345
- link RHip: mass 0.049473 -> 0.076
- link RTibia: mass 0.081897 -> 0.13355
- link base_link: mass 0.275 -> 0.431

Commit message: updated legs mass

File: test_legs_urdf/urdf/test_legs_urdf.urdf (robot description, URDF)
Before this commit: robot test_legs_urdf, 13 links, 12 joints
Links:
- link LLeg: mass 0.013241 -> 0.01406
- link RLeg: mass 0.013241 -> 0.01406
